File: ThumbsUp.sch (KiCad schematic (older format))
At the start: 159 parts, among them J19 52559-1233, J32 Battery, SW2 SW_DIP_x01, U1 ProMicro

Commit message: Replaced the switch footprint
Parts:
- MX1, MX10, MX11, MX12, MX13, MX14, MX15, MX16, MX17, MX18, MX19, MX2, MX20, MX21, MX22, MX23, MX24, MX25, MX26, MX27, MX28, MX29, MX3, MX30, MX31, MX32, MX33, MX34, MX35, MX36, MX37, MX38, MX39, MX4, MX40, MX41, MX42, MX43, MX44, MX45, MX46, MX47, MX48, MX49, MX5, MX50, MX51, MX52, MX53, MX54, MX55, MX56, MX57, MX58, MX6, MX7, MX8, MX9: footprint keyswitches:Kailh_socket_PG1350_optional -> keyswitches:PG1350_GLv2

Commit message: Wired Level 2.
Connections:
- net GND: now also JM11.1 (Pin_1)
- net L1GND: now also JF11.1 (Pin_1)
- net at D14.2 (A), MX10.2 (ROW): no longer JM11.1 (Pin_1)
- no-connect marks 14 -> 13
Changed lines of the file:
@@
 Wire Wire Line
 	2050 10850 2150 10850
-NoConn ~ 1850 10850
 Wire Wire Line
 	2150 11400 2050 11400
@@
 Wire Wire Line
 	3600 1200 3600 1100
-Wire Wire Line
-	1850 11400 1500 11400
-Wire Wire Line
-	1500 11400 1500 9450
-Wire Wire Line
-	1500 9450 2650 9450
-Connection ~ 2650 9450
 Text GLabel 4300 2850 2    50   Input ~ 0
 ROWR0
@@
 	0    -1   1    0
 $EndComp
+Wire Wire Line
+	1850 10850 1950 10850
+Connection ~ 1950 10850
+Wire Wire Line
+	1850 11400 1950 11400
+Connection ~ 1950 11400
 $EndSCHEMATC
