File: ThumbsUp.kicad_pcb (KiCad board)
At the start: 2 copper layers, 280.6 x 508.6 mm, 159 parts, among them J19 52559-1233, J32 Battery, SW2 SW_DIP_x01, U1 ProMicro

Commit message: Replaced the switch footprint
Parts:
- MX1, MX10, MX11, MX12, MX13, MX14, MX15, MX16, MX17, MX18, MX19, MX2, MX20, MX21, MX22, MX23, MX24, MX25, MX26, MX27, MX28, MX29, MX3, MX30, MX31, MX32, MX33, MX34, MX35, MX36, MX37, MX38, MX39, MX4, MX40, MX41, MX42, MX43, MX44, MX45, MX46, MX47, MX48, MX49, MX5, MX50, MX51, MX52, MX53, MX54, MX55, MX56, MX57, MX58, MX6, MX7, MX8, MX9: footprint keyswitches:Kailh_socket_PG1350_optional -> keyswitches:PG1350_GLv2

Commit message: Retraced the lower board
Routing:
- net Net-(JF33-Pad1): track 139.0 -> 152.3 mm, vias 0 -> 1
- net Net-(JF20-Pad2): track 140.2 -> 153.0 mm, vias 0 -> 1
- net Net-(JF20-Pad4): track 94.8 -> 106.5 mm
- net Net-(JF22-Pad4): track 95.2 -> 83.8 mm, vias 0 -> 1
- net Net-(JF31-Pad2): track 95.9 -> 84.7 mm, vias 0 -> 1
- net Net-(JF31-Pad3): track 72.9 -> 61.8 mm, vias 0 -> 1
- net Net-(JF21-Pad3): track 71.6 -> 61.0 mm, vias 0 -> 1
- net Net-(JF22-Pad3): track 71.2 -> 61.0 mm, vias 0 -> 1
- net Net-(JF20-Pad3): track 117.4 -> 127.2 mm, vias 0 -> 1
- net Net-(JF23-Pad1): track 108.7 -> 99.3 mm, vias 0 -> 1
- net Net-(JF21-Pad4): track 93.5 -> 84.2 mm, vias 0 -> 1
- net Net-(JF22-Pad2): track 51.9 -> 42.9 mm, vias 0 -> 1
- net Net-(JF28-Pad2): track 74.1 -> 83.1 mm, vias 0 -> 1
- net Net-(JF23-Pad3): track 81.6 -> 72.7 mm, vias 0 -> 1
- net Net-(JF21-Pad1): track 41.2 -> 32.4 mm, vias 0 -> 1
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
Commit message: Redefined the layout, checked in before splitting the layers.
Parts:
- moved JM45 550.4 mm to (-397.0, 99.0)
- moved JM5 549.1 mm to (-256.5, 114.1)
- moved JM13 541.2 mm to (-323.0, 64.5)
- moved MX53 540.5 mm to (-288.2, 127.4), turned to 37 degrees
- moved MX26 540.5 mm to (-257.8, 104.5), turned to 37 degrees
- moved MX30 540.5 mm to (-273.0, 115.9), turned to 37 degrees
- moved J19 536.1 mm to (-297.8, 111.6)
- moved MX18 533.7 mm to (-372.8, 115.9), turned to 323 degrees
- moved MX22 533.7 mm to (-388.0, 104.5), turned to 323 degrees
- moved MX51 533.7 mm to (-357.6, 127.4), turned to 323 degrees
- moved JM43 530.2 mm to (-381.9, 119.7)
- moved JM17 503.3 mm to (-250.0, 99.9)
- moved JF45 494.1 mm to (-397.0, 99.0)
- moved JF33 488.8 mm to (-271.7, 125.6), turned to 307 degrees
- moved JF28 486.0 mm to (-269.4, 76.5)
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Routing:
- net GND: track 420.6 -> 0.00 mm, vias 1 -> 0
- net COL5: track 415.7 -> 0.00 mm, vias 6 -> 0
- net COL4: track 366.7 -> 0.00 mm, vias 5 -> 0
- net COL2: track 359.7 -> 0.00 mm, vias 5 -> 0
- net COL3: track 336.2 -> 0.00 mm, vias 8 -> 0
- net COL1: track 232.3 -> 0.00 mm, vias 2 -> 0
- net COL0: track 178.6 -> 0.00 mm, vias 2 -> 0
- net Net-(JF33-Pad4): track 177.4 -> 0.00 mm, vias 1 -> 0
- net Net-(JF20-Pad1): track 170.0 -> 0.00 mm, vias 1 -> 0
- net Net-(JF33-Pad3): track 158.5 -> 0.00 mm, vias 1 -> 0
- net Net-(JF20-Pad2): track 153.0 -> 0.00 mm, vias 1 -> 0
- net Net-(JF33-Pad1): track 152.3 -> 0.00 mm, vias 1 -> 0
- net ROWR4: track 145.7 -> 0.00 mm
- net Net-(JF33-Pad2): track 144.6 -> 0.00 mm, vias 1 -> 0
- net SDA: track 131.5 -> 0.00 mm, vias 1 -> 0
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Other:
- board size 280.6 x 508.6 mm -> 282 x 148.4 mm

Commit message: Split the PCBs
Parts:
- moved D23 645.4 mm to (-308.6, 272.3)
- moved D25 645.4 mm to (-308.6, 304.4)
- moved D27 645.4 mm to (-308.6, 301.9)
- moved D34 645.4 mm to (-308.6, 286.9)
- moved D52 645.4 mm to (-308.6, 269.9)
- moved D55 645.4 mm to (-308.6, 281.9)
- moved D56 645.4 mm to (-308.6, 279.6)
- moved D58 645.4 mm to (-308.6, 274.8)
- moved D24 645.4 mm to (-308.6, 296.9)
- moved D26 645.4 mm to (-308.6, 299.4)
- moved D31 645.4 mm to (-308.6, 294.4)
- moved D32 645.4 mm to (-308.6, 291.9)
- moved D33 645.4 mm to (-308.6, 289.4)
- moved D54 645.4 mm to (-308.6, 284.4)
- moved D57 645.4 mm to (-308.6, 277.1)
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Routing:
- net L3GND: track 7.62 -> 0.00 mm
- removed copper zone on B.Cu, net L1GND
Other:
- board size 282 x 148.4 mm -> 282 x 464.4 mm
- board text added: "ThumbsUp! v8 Choc/Gat Low Profile, ProMicro u/ak66666 Oct 01, 2023"
- board text removed: "ThumbsUp! v5 MX/ALPS ProMicro u/ak66666 May 22, 2023"

Commit message: Started tracing the secoh
Parts:
- moved D30 19.2 mm to (-281.7, 308.6), turned to 270 degrees
- moved D29 14.9 mm to (-278.9, 308.6), turned to 270 degrees
- moved D45 3.22 mm to (-336.4, 284.6)
- moved D48 3.22 mm to (-336.4, 277.1)
- moved D15 3.22 mm to (-336.4, 292.1)
- moved D16 3.22 mm to (-336.4, 294.6)
- moved D20 3.22 mm to (-336.4, 272.2)
- moved D21 3.22 mm to (-336.4, 287.1)
- moved D46 3.22 mm to (-336.4, 282.1)
- moved D47 3.22 mm to (-336.4, 279.6)
- moved D49 3.22 mm to (-336.4, 289.6)
- moved D50 3.22 mm to (-336.4, 274.7)
- moved D28 2.00 mm to (-275.9, 299.4)
- moved D35 2.00 mm to (-289.9, 299.4)
- moved D36 2.00 mm to (-292.7, 299.4)
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Routing:
- net COL4: track 0.00 -> 162.3 mm
- net COL5: track 0.00 -> 128.0 mm
- net Net-(D27-Pad2): track 0.00 -> 100.9 mm, vias 0 -> 2
- net Net-(D26-Pad2): track 0.00 -> 93.1 mm, vias 0 -> 2
- net Net-(D54-Pad2): track 0.00 -> 91.5 mm, vias 0 -> 2
- net Net-(D55-Pad2): track 0.00 -> 86.7 mm, vias 0 -> 1
- net Net-(D45-Pad2): track 0.00 -> 86.6 mm, vias 0 -> 1
- net Net-(D31-Pad2): track 0.00 -> 84.9 mm, vias 0 -> 1
- net Net-(D49-Pad2): track 0.00 -> 83.6 mm, vias 0 -> 2
- net Net-(D56-Pad2): track 0.00 -> 82.3 mm, vias 0 -> 1
- net Net-(D46-Pad2): track 0.00 -> 81.3 mm, vias 0 -> 1
- net Net-(D44-Pad2): track 0.00 -> 81.3 mm, vias 0 -> 2
- net Net-(D32-Pad2): track 0.00 -> 80.2 mm, vias 0 -> 1
- net Net-(D4-Pad2): track 0.00 -> 79.8 mm, vias 0 -> 1
- net Net-(D57-Pad2): track 0.00 -> 78.0 mm, vias 0 -> 1
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
Commit message: Fixed and moved the cross board connectors.
Parts:
- removed the JF33 at (-271.6, 314.4)
- added JF33: Conn_01x04_Female, Connector_PinSocket_2.54mm:PinSocket_1x04_P2.54mm_Vertical, F.Cu at (-283.4, 511.8)
- added JF33: Conn_01x04_Female, Connector_PinSocket_2.54mm:PinSocket_1x04_P2.54mm_Vertical, F.Cu at (-283.5, 323.0)
- moved JM33 197.7 mm to (-283.5, 323.0)
- moved JM23 196.6 mm to (-362.5, 323.0)
- moved JF23 196.6 mm to (-362.4, 511.7)
- moved JM5 188.7 mm to (-256.6, 114.2)
- moved JF5 188.7 mm to (-256.4, 302.9)
- moved JF43 188.5 mm to (-381.4, 308.8)
- moved JM43 188.5 mm to (-381.5, 120.0)
- moved JM17 58.3 mm to (-298.0, 133.0)
- moved JF17 58.3 mm to (-297.9, 321.8)
- moved JF45 57.5 mm to (-347.9, 321.8)
- moved JM45 57.5 mm to (-348.0, 133.0)
- moved R1 12.6 mm to (-304.2, 315.6)
- moved R2 12.6 mm to (-302.2, 315.6)
- moved JM11 0.51 mm to (-433.9, 272.3)
- moved JF11 0.51 mm to (-433.8, 461.1)
Connections:
- JF11 pad 2: L1GND -> (no net)
- JF11 pad 3: L1GND -> (no net)
- JF11 pad 4: L1GND -> (no net)
- JF17 pad 1: VCC -> (no net)
- JF17 pad 2: SDA -> (no net)
- JF17 pad 3: SCL -> (no net)
- JF17 pad 4: GND -> (no net)
- JF23 pad 1: Net-(JF23-Pad1) -> (no net)
- JF23 pad 2: Net-(JF23-Pad2) -> (no net)
- JF23 pad 3: Net-(JF23-Pad3) -> (no net)
- JF23 pad 4: Net-(JF23-Pad4) -> (no net)
- JF43 pad 1: COL4 -> (no net)
- JF43 pad 2: Net-(D18-Pad2) -> (no net)
- JF43 pad 3: Net-(D19-Pad2) -> (no net)
- JF43 pad 4: COL5 -> (no net)
- JF45 pad 1: COL1 -> (no net)
- JF45 pad 2: Net-(D53-Pad2) -> (no net)
- JF45 pad 3: Net-(D51-Pad2) -> (no net)
- JF45 pad 4: COL1 -> (no net)
- JF5 pad 1: COL5 -> (no net)
- JF5 pad 2: Net-(D29-Pad2) -> (no net)
- JF5 pad 3: Net-(D30-Pad2) -> (no net)
- JF5 pad 4: COL4 -> (no net)
- JM11 pad 1: Net-(D14-Pad2) -> (no net)
- JM11 pad 2: GND -> (no net)
- JM11 pad 3: GND -> (no net)
- JM11 pad 4: GND -> (no net)
- JM23 pad 1: Net-(D12-Pad2) -> (no net)
- JM23 pad 2: Net-(D11-Pad2) -> (no net)
- JM23 pad 3: Net-(D10-Pad2) -> (no net)
- JM23 pad 4: Net-(D9-Pad2) -> (no net)
- JM33 pad 1: COL3 -> (no net)
- JM33 pad 2: COL2 -> (no net)
- JM33 pad 3: COL1 -> (no net)
- JM33 pad 4: COL0 -> (no net)
- JM43 pad 1: Net-(JM43-Pad1) -> (no net)
- JM43 pad 2: Net-(JM43-Pad2) -> (no net)
- JM43 pad 3: Net-(JM43-Pad3) -> (no net)
- JM43 pad 4: Net-(JM43-Pad4) -> (no net)
- JM45 pad 1: Net-(JM45-Pad1) -> (no net)
- JM45 pad 2: Net-(JM45-Pad2) -> (no net)
- JM45 pad 3: Net-(JM45-Pad3) -> (no net)
- JM45 pad 4: Net-(JM45-Pad4) -> (no net)
- JM5 pad 1: Net-(JM5-Pad1) -> (no net)
- JM5 pad 2: Net-(JM5-Pad2) -> (no net)
- JM5 pad 3: Net-(JM5-Pad3) -> (no net)
- JM5 pad 4: Net-(JM5-Pad4) -> (no net)
Routing:
- net GND: track 14.1 -> 8.57 mm
- net (no net): track 0.00 -> 5.50 mm
Other:
- outline, holes or cut-outs redrawn

Commit message: Wired Level 2.
Parts:
- removed the JF33 at (-283.5, 323.0)
- moved D30 19.2 mm to (-264.9, 299.4), turned to 90 degrees
- moved D29 14.5 mm to (-267.7, 299.4), turned to 90 degrees
- moved SW2 5.96 mm to (-330.6, 324.6), turned to 0 degrees
- moved S1 5.64 mm to (-311.9, 325.7), turned to 0 degrees
- moved R1 2.40 mm to (-304.4, 318.1), turned to 270 degrees
- moved R2 2.39 mm to (-302.4, 318.0), turned to 90 degrees
Connections:
- JF11 pad 1: (no net) -> L1GND
- JF11 pad 2: (no net) -> L1GND
- JF11 pad 3: (no net) -> L1GND
- JF11 pad 4: (no net) -> L1GND
- JF17 pad 1: (no net) -> VCC
- JF17 pad 2: (no net) -> SDA
- JF17 pad 3: (no net) -> SCL
- JF17 pad 4: (no net) -> GND
- JF23 pad 1: (no net) -> Net-(JF23-Pad1)
- JF23 pad 2: (no net) -> Net-(JF23-Pad2)
- JF23 pad 3: (no net) -> Net-(JF23-Pad3)
- JF23 pad 4: (no net) -> Net-(JF23-Pad4)
- JF33 pad 1: (no net) -> Net-(JF33-Pad1)
- JF33 pad 2: (no net) -> Net-(JF33-Pad2)
- JF33 pad 3: (no net) -> Net-(JF33-Pad3)
- JF33 pad 4: (no net) -> Net-(JF33-Pad4)
- JF43 pad 1: (no net) -> COL4
- JF43 pad 2: (no net) -> Net-(D18-Pad2)
- JF43 pad 3: (no net) -> Net-(D19-Pad2)
- JF43 pad 4: (no net) -> COL5
- JF45 pad 1: (no net) -> COL1
- JF45 pad 2: (no net) -> Net-(D53-Pad2)
- JF45 pad 3: (no net) -> Net-(D51-Pad2)
- JF45 pad 4: (no net) -> COL1
- JF5 pad 1: (no net) -> COL5
- JF5 pad 2: (no net) -> Net-(D29-Pad2)
- JF5 pad 3: (no net) -> Net-(D30-Pad2)
- JF5 pad 4: (no net) -> COL4
- JM11 pad 1: (no net) -> GND
- JM11 pad 2: (no net) -> GND
- JM11 pad 3: (no net) -> GND
- JM11 pad 4: (no net) -> GND
- JM23 pad 1: (no net) -> Net-(D12-Pad2)
- JM23 pad 2: (no net) -> Net-(D11-Pad2)
- JM23 pad 3: (no net) -> Net-(D10-Pad2)
- JM23 pad 4: (no net) -> Net-(D9-Pad2)
- JM33 pad 1: (no net) -> COL3
- JM33 pad 2: (no net) -> COL2
- JM33 pad 3: (no net) -> COL1
- JM33 pad 4: (no net) -> COL0
- JM43 pad 1: (no net) -> Net-(JM43-Pad1)
- JM43 pad 2: (no net) -> Net-(JM43-Pad2)
- JM43 pad 3: (no net) -> Net-(JM43-Pad3)
- JM43 pad 4: (no net) -> Net-(JM43-Pad4)
- JM45 pad 1: (no net) -> Net-(JM45-Pad1)
- JM45 pad 2: (no net) -> Net-(JM45-Pad2)
- JM45 pad 3: (no net) -> Net-(JM45-Pad3)
- JM45 pad 4: (no net) -> Net-(JM45-Pad4)
- JM5 pad 1: (no net) -> Net-(JM5-Pad1)
- JM5 pad 2: (no net) -> Net-(JM5-Pad2)
- JM5 pad 3: (no net) -> Net-(JM5-Pad3)
- JM5 pad 4: (no net) -> Net-(JM5-Pad4)
Routing:
- net GND: track 8.57 -> 391.5 mm, vias 0 -> 2
- net COL2: track 24.2 -> 397.0 mm, vias 0 -> 3
- net COL3: track 25.3 -> 358.5 mm, vias 0 -> 5
- net COL5: track 128.0 -> 392.7 mm, vias 0 -> 12
- net COL4: track 162.3 -> 396.8 mm, vias 0 -> 4
- net COL1: track 0.00 -> 193.7 mm, vias 0 -> 3
- net COL0: track 0.00 -> 153.6 mm, vias 0 -> 2
- net ROWR4: track 0.00 -> 126.3 mm
- net ROWL4: track 0.00 -> 110.7 mm, vias 0 -> 1
- net ROWL3: track 0.00 -> 108.8 mm, vias 0 -> 1
- net SDA: track 0.00 -> 97.1 mm, vias 0 -> 1
- net SCL: track 0.00 -> 95.9 mm, vias 0 -> 1
- net +BATT: track 0.00 -> 84.2 mm
- net RST: track 0.00 -> 82.7 mm
- net VCC: track 0.00 -> 81.8 mm, vias 0 -> 1
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
Commit message: Wired all levels
Routing:
- net Net-(JF33-Pad4): track 0.00 -> 213.8 mm, vias 0 -> 1
- net Net-(JF33-Pad3): track 0.00 -> 191.4 mm, vias 0 -> 1
- net Net-(JF20-Pad1): track 0.00 -> 178.9 mm, vias 0 -> 1
- net Net-(JF33-Pad2): track 0.00 -> 169.4 mm, vias 0 -> 1
- net Net-(JF20-Pad2): track 0.00 -> 160.0 mm, vias 0 -> 1
- net Net-(JF33-Pad1): track 0.00 -> 150.6 mm, vias 0 -> 1
- net Net-(JF23-Pad1): track 0.00 -> 132.7 mm, vias 0 -> 1
- net Net-(JF20-Pad3): track 0.00 -> 131.7 mm, vias 0 -> 1
- net Net-(JF28-Pad1): track 0.00 -> 122.7 mm, vias 0 -> 1
- net Net-(JF23-Pad2): track 0.00 -> 113.9 mm, vias 0 -> 1
- net Net-(JF31-Pad1): track 0.00 -> 108.9 mm, vias 0 -> 1
- net Net-(JF20-Pad4): track 0.00 -> 108.6 mm, vias 0 -> 1
- net Net-(JF30-Pad1): track 0.00 -> 107.8 mm, vias 0 -> 1
- net Net-(JF29-Pad1): track 0.00 -> 107.2 mm, vias 0 -> 1
- net Net-(JF3-Pad1): track 0.00 -> 96.3 mm, vias 0 -> 1
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- added copper zone on B.Cu, net L1GND
Other:
- board text added: "QMK: "matrix_pins": { "cols": ["C6", "D4", "D2", "D3", "B6", "D7"], "rows": ["B4", "F6", "E6", "F7", "B5", "B1", "F4", "B3", "F5", "B2"]},"
- board text added: "ThumbsUp! v8 ProMicro Kailh Choc/Gat Low Profile Hot-Swap Sockets u/ak66666, Oct 01, 2023"
- board text removed: "QMK: "matrix_pins": { "cols": ["C6", "D4", "D2", "D3", "B6", "D7"], "rows": ["B4", "F6", "E6", "F7", "B5", "B1", "F4", "B3", "F5", "B2"] },"
- board text removed: "ThumbsUp! v8 Choc/Gat Low Profile, ProMicro u/ak66666 Oct 01, 2023"
